Commit message: Created new Xiao Serial Bridge IMU module

File: slam_ros2_ws/src/robot_slam/urdf/robot.urdf.xacro (robot description, xacro)
@@ -5,8 +5,8 @@
   <joint name="lidar_joint" type="fixed">
     <parent link="base_link"/>
-    <child link="laser_frame"/>
-    <origin xyz="0.1 0.0 0.2" rpy="0 0 0"/>  <!-- adjust to your mount -->
+    <child link="laser"/>
+    <origin xyz="0.1 0.0 0.2" rpy="0 0 0"/>
   </joint>
-  <link name="laser_frame"/>
+  <link name="laser"/>
   <!-- OAK-D Lite -->
   <joint name="camera_joint" type="fixed">
@@ -19,7 +19,7 @@
   <joint name="imu_joint" type="fixed">
     <parent link="base_link"/>
-    <child link="imu_link"/>
+    <child link="base_imu_link"/>
     <origin xyz="0.0 0.0 0.1" rpy="0 0 0"/>
   </joint>
-  <link name="imu_link"/>
+  <link name="base_imu_link"/>
 </robot>
